File: hardware/v1.2_neo/angle_detect.kicad_pcb (KiCad board)
At the start: 2 copper layers, 82.9 x 42.2 mm, 54 parts, among them J1 Conn_01x07, J2 Conn_01x07, J3 USB_C_Receptacle_USB2.0, J4 IIC_OLED, J5 SWD, J6 Conn_01x03, SW1 NRST_BUTTON, SW2 USER_BUTTON, U1 STM32G474RETx, U2 MPU-9250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

Commit message: fake
Parts:
- U2, U3: footprint Sensor_Motion:InvenSense_QFN-24_3x3mm_P0.4mm -> Package_DFN_QFN:QFN-24-1EP_3x3mm_P0.4mm_EP1.75x1.6mm
- moved J4 7.62 mm to (78.0, 142.5), turned to 180 degrees
Routing:
- net GND: track 54.7 -> 58.8 mm
- net /OLED_SDA: track 10.9 -> 8.69 mm, vias 1 -> 0
- net /GND_B: track 21.2 -> 22.7 mm
- net +3.3V: track 149.2 -> 150.2 mm
- net /OLED_SCL: track 8.53 -> 7.84 mm, vias 1 -> 0
Other:
- board text added: "CLK"
- board text added: "DIO"
- board text added: "GND"
- board text added: "VCC"
