File: hardware/v1.2_neo/angle_detect.kicad_sch (KiCad schematic)
At the start: 54 parts, among them J1 Conn_01x07, J2 Conn_01x07, J3 USB_C_Receptacle_USB2.0, J4 IIC_OLED, J5 SWD, J6 Conn_01x03, SW1 NRST_BUTTON, SW2 USER_BUTTON, U1 STM32G474RETx, U2 MPU-9250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

Commit message: fake
Parts:
- U2, U3: footprint Sensor_Motion:InvenSense_QFN-24_3x3mm_P0.4mm -> Package_DFN_QFN:QFN-24-1EP_3x3mm_P0.4mm_EP1.75x1.6mm
Connections:
- net +3.3V: no longer J4.3 (Pin_3)
Changed lines of the file:
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@@
-    (stroke (width 0) (type default))
-  )
-  (wire (pts (xy 145.288 186.436) (xy 151.384 186.436))
     (stroke (width 0) (type default))
   )
@@
       (effects (font (size 1.27 1.27)) (justify left))
     )
-    (property "Footprint" "Sensor_Motion:InvenSense_QFN-24_3x3mm_P0.4mm" (at 233.172 132.334 0)
+    (property "Footprint" "Package_DFN_QFN:QFN-24-1EP_3x3mm_P0.4mm_EP1.75x1.6mm" (at 233.172 132.334 0)
       (effects (font (size 1.27 1.27)) hide)
     )
@@
       (effects (font (size 1.27 1.27)) (justify left))
     )
-    (property "Footprint" "Sensor_Motion:InvenSense_QFN-24_3x3mm_P0.4mm" (at 232.156 69.85 0)
-      (effects (font (size 1.27 1.27)) hide)
-    )
+    (property "Footprint" "Package_DFN_QFN:QFN-24-1EP_3x3mm_P0.4mm_EP1.75x1.6mm" (at 232.156 69.85 0)
+      (effects (font (size 1.27 1.27)) hide)
+    )
